Commit message: Add pose_frame link

File: realsense2_description/urdf/_t265.urdf.xacro (robot description, xacro)
@@ -23,7 +23,13 @@
     </material>
     <!-- camera body, with origin at camera_link -->
-    <joint name="${name}_pose_joint" type="fixed">
+    <joint name="${name}_pose_frame_joint" type="fixed">
       <xacro:insert_block name="origin" />
       <parent link="${parent}"/>
+      <child link="${name}_pose_frame" />
+    </joint>
+    <link name="${name}_pose_frame"/>
+    <joint name="${name}_pose_joint" type="fixed">
+      <origin xyz="0 0 0" rpy="0 0 0"/>
+      <parent link="${name}_pose_frame"/>
       <child link="${name}_link" />
     </joint>

Commit message: Add transform between pose_frame and camera link for image orientation

File: realsense2_description/urdf/_t265.urdf.xacro (robot description, xacro)
@@ -30,5 +30,5 @@
     <link name="${name}_pose_frame"/>
     <joint name="${name}_pose_joint" type="fixed">
-      <origin xyz="0 0 0" rpy="0 0 0"/>
+      <origin xyz="0 0 0" rpy="${90 * deg_to_rad} 0 ${-90 * deg_to_rad}"/>
       <parent link="${name}_pose_frame"/>
       <child link="${name}_link" />
